File: pcb/eink-environment-clock/eink-environment-clock.kicad_pcb (KiCad board)
At the start: 2 copper layers, 91.8 x 37.5 mm, 23 parts, among them J1 J1_PWR, J2 J2_EPD, U1 U1_ESP32C3, U2 U2_BME280, U3 RTC_DS3231, U4 U4_MH-Z19B

Commit message: feat(pcb): Add images and update R8
Parts:
- R8: value R8_UART_TX_10k -> R8_UART_TX_470R
Changed lines of the file:
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@@
 			)
 		)
-		(property "Value" "R8_UART_TX_10k"
+		(property "Value" "R8_UART_TX_470R"
 			(at 3.81 2.37 0)
 			(layer "F.Fab")
